File: pcb/unix-wall-clock.kicad_sch (KiCad schematic)
At the start: 8 parts

Commit message: add video
Parts:
- C1: renamed from U; value (none) -> 10uF; footprint (none) -> Capacitor_SMD:C_0603_1608Metric
- J1, J2: renamed from U; value (none) -> Conn_01x08_Female; footprint (none) -> Connector_PinSocket_2.54mm:PinSocket_1x08_P2.54mm_Vertical
- J3, J4: renamed from U; value (none) -> Conn_01x07_Female; footprint (none) -> Connector_PinSocket_2.54mm:PinSocket_1x07_P2.54mm_Vertical
- R1: renamed from U; value (none) -> 2.7K; footprint (none) -> Resistor_SMD:R_0603_1608Metric
- R2: renamed from U; value (none) -> DNP; footprint (none) -> Resistor_SMD:R_0603_1608Metric
- U1: renamed from U; value (none) -> STP16CP05; footprint (none) -> Package_SO:QSOP-24_3.9x8.7mm_P0.635mm
